File: Kicad/Token.sch (KiCad schematic (older format))
At the start: 10 parts

Commit message: Added folder and first project for ESP8266
Parts:
- DS?: symbol LCD-016N002L -> LCD-016N002L-RESCUE-Token
Changed lines of the file:
@@
 EESchema Schematic File Version 2
+LIBS:Token-rescue
 LIBS:power
 LIBS:device
@@
 LIBS:valves
 LIBS:stm32
+LIBS:Token-cache
 EELAYER 25 0
 EELAYER END
@@
 	3400 2700 3300 2700
 $Comp
-L LCD-016N002L DS?
+L LCD-016N002L-RESCUE-Token DS?
 U 1 1 581C7047
 P 1450 2750
